Commit message: Phase 2-C: slam_toolbox + my_map

File: install/amr_description/share/amr_description/urdf/amr_robot.urdf.xacro (robot description, xacro)
@@ -1,187 +1 @@
-<?xml version="1.0"?>
-<robot name="visual_amr" xmlns:xacro="http://www.ros.org/wiki/xacro" xmlns:gz="http://gazebosim.org/schema">
-  <material name="silver"><color rgba="0.700 0.700 0.700 1.000"/></material>
-  <material name="blue"><color rgba="0.0 0.0 0.8 1.0"/></material>
-  <material name="black"><color rgba="0.1 0.1 0.1 1.0"/></material>
-  <link name="base_footprint"/>
-  <joint name="base_joint" type="fixed">
-    <parent link="base_footprint"/>
-    <child link="base_link"/>
-    <origin xyz="0 0 0.1" rpy="0 0 0"/>
-  </joint>
-  <link name="base_link">
-    <visual>
-      <geometry><box size="0.4 0.4 0.15"/></geometry>
-      <material name="silver"/>
-    </visual>
-    <collision>
-      <geometry><box size="0.4 0.4 0.15"/></geometry>
-    </collision>
-    <inertial>
-      <origin xyz="0 0 0" rpy="0 0 0"/>
-      <mass value="10.0"/>
-      <inertia ixx="${(1/12) * 10.0 * (0.4*0.4 + 0.15*0.15)}" ixy="0.0" ixz="0.0"
-               iyy="${(1/12) * 10.0 * (0.4*0.4 + 0.15*0.15)}" iyz="0.0"
-               izz="${(1/12) * 10.0 * (0.4*0.4 + 0.4*0.4)}"/>
-    </inertial>
-  </link>
-  <!-- Include and invoke 4-wheel omni base macro -->
-  <xacro:include filename="base_omni_4wheel.xacro"/>
-  <xacro:base_omni_4wheel/>
-  <joint name="oak_d_joint" type="fixed">
-    <parent link="base_link"/>
-    <child link="oak_d_link"/>
-    <origin xyz="0.18 0 0.1" rpy="0 0.26 0"/>
-  </joint>
-  <link name="oak_d_link">
-    <visual>
-      <geometry><box size="0.03 0.1 0.03"/></geometry>
-      <material name="black"/>
-    </visual>
-    <inertial>
-      <origin xyz="0 0 0" rpy="0 0 0"/>
-      <mass value="0.15"/>
-      <inertia ixx="${(1/12) * 0.15 * (0.1*0.1 + 0.03*0.03)}" ixy="0.0" ixz="0.0"
-               iyy="${(1/12) * 0.15 * (0.03*0.03 + 0.03*0.03)}" iyz="0.0"
-               izz="${(1/12) * 0.15 * (0.03*0.03 + 0.1*0.1)}"/>
-    </inertial>
-  </link>
-  <joint name="arm_base_joint" type="fixed">
-    <parent link="base_link"/>
-    <child link="arm_base_link"/>
-    <origin xyz="0.1 0 0.075" rpy="0 0 0"/>
-  </joint>
-  <link name="arm_base_link">
-    <visual>
-      <geometry><cylinder radius="0.05" length="0.04"/></geometry>
-      <material name="blue"/>
-    </visual>
-    <inertial>
-      <origin xyz="0 0 0" rpy="0 0 0"/>
-      <mass value="0.5"/>
-      <inertia ixx="${(1/12) * 0.5 * (3*0.05*0.05 + 0.04*0.04)}" ixy="0.0" ixz="0.0"
-               iyy="${(1/12) * 0.5 * (3*0.05*0.05 + 0.04*0.04)}" iyz="0.0"
-               izz="${0.5 * 0.5 * 0.05 * 0.05}"/>
-    </inertial>
-  </link>
-  <!-- Include and invoke SO-101 arm macro -->
-  <xacro:include filename="so101_arm.xacro"/>
-  <xacro:so101_arm/>
-  <!-- Include and invoke parallel gripper macro -->
-  <xacro:include filename="gripper.xacro"/>
-  <xacro:so101_gripper/>
-  <!-- Self collision settings for base_link -->
-  <gazebo reference="base_link">
-    <self_collision>true</self_collision>
-  </gazebo>
-  <!-- ros2_control configuration for arm and gripper -->
-  <ros2_control name="amr_robot_system" type="system">
-    <hardware>
-      <plugin>gz_ros2_control/GazeboSimSystem</plugin>
-    </hardware>
-    <!-- Arm Joints -->
-    <joint name="joint1">
-      <command_interface name="position"/>
-      <state_interface name="position">
-        <param name="initial_value">0.0</param>
-      </state_interface>
-      <state_interface name="velocity"/>
-    </joint>
-    <joint name="joint2">
-      <command_interface name="position"/>
-      <state_interface name="position">
-        <param name="initial_value">0.0</param>
-      </state_interface>
-      <state_interface name="velocity"/>
-    </joint>
-    <joint name="joint3">
-      <command_interface name="position"/>
-      <state_interface name="position">
-        <param name="initial_value">0.0</param>
-      </state_interface>
-      <state_interface name="velocity"/>
-    </joint>
-    <joint name="joint4">
-      <command_interface name="position"/>
-      <state_interface name="position">
-        <param name="initial_value">0.0</param>
-      </state_interface>
-      <state_interface name="velocity"/>
-    </joint>
-    <joint name="joint5">
-      <command_interface name="position"/>
-      <state_interface name="position">
-        <param name="initial_value">0.0</param>
-      </state_interface>
-      <state_interface name="velocity"/>
-    </joint>
-    <joint name="joint6">
-      <command_interface name="position"/>
-      <state_interface name="position">
-        <param name="initial_value">0.0</param>
-      </state_interface>
-      <state_interface name="velocity"/>
-    </joint>
-    <!-- Gripper Joints -->
-    <joint name="left_finger_joint">
-      <command_interface name="position"/>
-      <state_interface name="position">
-        <param name="initial_value">0.0</param>
-      </state_interface>
-      <state_interface name="velocity"/>
-    </joint>
-    <joint name="right_finger_joint">
-      <command_interface name="position"/>
-      <state_interface name="position">
-        <param name="initial_value">0.0</param>
-      </state_interface>
-      <state_interface name="velocity"/>
-    </joint>
-  </ros2_control>
-  <!-- Gazebo Sim ros2_control plugin -->
-  <gazebo>
-    <plugin filename="gz_ros2_control-system" name="gz_ros2_control::GazeboSimROS2ControlPlugin">
-      <parameters>$(find amr_description)/config/amr_controllers.yaml</parameters>
-      <hold_joints>false</hold_joints>
-    </plugin>
-  </gazebo>
-  <!-- IMU Sensor -->
-  <gazebo reference="base_link">
-    <sensor name="imu_sensor" type="imu">
-      <always_on>1</always_on>
-      <update_rate>50</update_rate>
-      <visualize>true</visualize>
-      <topic>imu</topic>
-    </sensor>
-  </gazebo>
-  <!-- OAK-D RGB-D Camera Sensor -->
-  <gazebo reference="oak_d_link">
-    <sensor name="oakd_camera" type="rgbd">
-      <always_on>1</always_on>
-      <update_rate>30</update_rate>
-      <camera>
-        <horizontal_fov>1.25</horizontal_fov>
-        <image>
-          <width>640</width>
-          <height>480</height>
-          <format>R8G8B8</format>
-        </image>
-        <clip>
-          <near>0.1</near>
-          <far>10.0</far>
-        </clip>
-      </camera>
-      <topic>camera</topic>
-    </sensor>
-  </gazebo>
-  <!-- Gazebo Sim Sensor Plugins -->
-  <gazebo>
-    <plugin filename="gz-sim-imu-system" name="gz::sim::systems::Imu">
-    </plugin>
-    <plugin filename="gz-sim-sensors-system" name="gz::sim::systems::Sensors">
-      <render_engine>ogre2</render_engine>
-    </plugin>
-    <plugin filename="gz-sim-joint-state-publisher-system" name="gz::sim::systems::JointStatePublisher">
-    </plugin>
-  </gazebo>
-</robot>
+/home/pakku/auto-trash-navigator/src/amr_description/urdf/amr_robot.urdf.xacro

File: install/amr_description/share/amr_description/urdf/base_omni_4wheel.xacro (robot description, xacro)
@@ -1,75 +1 @@
-<?xml version="1.0"?>
-<robot xmlns:xacro="http://www.ros.org/wiki/xacro" xmlns:gz="http://gazebosim.org/schema">
-  <!-- Macro for a single omni wheel -->
-  <xacro:macro name="omni_wheel" params="prefix x_reflect y_reflect fdir">
-    <joint name="${prefix}_wheel_joint" type="continuous">
-      <parent link="base_link"/>
-      <child link="${prefix}_wheel_link"/>
-      <origin xyz="${x_reflect * 0.15} ${y_reflect * 0.18} -0.05" rpy="0 0 ${(1 - y_reflect) * pi / 2}"/>
-      <axis xyz="0 ${y_reflect} 0"/>
-    </joint>
-    <link name="${prefix}_wheel_link">
-      <visual>
-        <origin xyz="0 0 0" rpy="${pi/2} 0 0"/>
-        <geometry>
-          <cylinder radius="0.05" length="0.04"/>
-        </geometry>
-        <material name="black"/>
-      </visual>
-      <collision>
-        <origin xyz="0 0 0" rpy="${pi/2} 0 0"/>
-        <geometry>
-          <cylinder radius="0.05" length="0.04"/>
-        </geometry>
-      </collision>
-      <inertial>
-        <origin xyz="0 0 0" rpy="${pi/2} 0 0"/>
-        <mass value="0.2"/>
-        <inertia ixx="${(1/12) * 0.2 * (3 * 0.05 * 0.05 + 0.04 * 0.04)}" ixy="0.0" ixz="0.0"
-                 iyy="${(1/12) * 0.2 * (3 * 0.05 * 0.05 + 0.04 * 0.04)}" iyz="0.0"
-                 izz="${0.5 * 0.2 * 0.05 * 0.05}"/>
-      </inertial>
-    </link>
-    <gazebo reference="${prefix}_wheel_link">
-      <collision>
-        <surface>
-          <friction>
-            <ode>
-              <mu>1.0</mu>
-              <mu2>0.0</mu2>
-              <fdir1 gz:expressed_in="base_footprint">${fdir}</fdir1>
-            </ode>
-          </friction>
-        </surface>
-      </collision>
-    </gazebo>
-  </xacro:macro>
-  <!-- Macro to add 4 omni wheels -->
-  <xacro:macro name="base_omni_4wheel">
-    <xacro:omni_wheel prefix="front_left" x_reflect="1" y_reflect="1" fdir="1 -1 0"/>
-    <xacro:omni_wheel prefix="front_right" x_reflect="1" y_reflect="-1" fdir="-1 -1 0"/>
-    <xacro:omni_wheel prefix="rear_left" x_reflect="-1" y_reflect="1" fdir="1 1 0"/>
-    <xacro:omni_wheel prefix="rear_right" x_reflect="-1" y_reflect="-1" fdir="-1 1 0"/>
-    <!-- Mecanum Drive Plugin for Gazebo Sim -->
-    <gazebo>
-      <plugin
-        filename="gz-sim-mecanum-drive-system"
-        name="gz::sim::systems::MecanumDrive">
-        <front_left_joint>front_left_wheel_joint</front_left_joint>
-        <front_right_joint>front_right_wheel_joint</front_right_joint>
-        <back_left_joint>rear_left_wheel_joint</back_left_joint>
-        <back_right_joint>rear_right_wheel_joint</back_right_joint>
-        <wheel_separation>0.36</wheel_separation>
-        <wheel_base>0.30</wheel_base>
-        <wheel_radius>0.05</wheel_radius>
-        <topic>/cmd_vel</topic>
-        <odom_topic>/odom</odom_topic>
-        <frame_id>odom</frame_id>
-        <child_frame_id>base_footprint</child_frame_id>
-        <publish_odom>true</publish_odom>
-        <publish_odom_tf>false</publish_odom_tf>
-        <odom_publish_frequency>50</odom_publish_frequency>
-      </plugin>
-    </gazebo>
-  </xacro:macro>
-</robot>
+/home/pakku/auto-trash-navigator/src/amr_description/urdf/base_omni_4wheel.xacro

File: install/amr_description/share/amr_description/urdf/gripper.xacro (robot description, xacro)
@@ -1,100 +1 @@
-<?xml version="1.0"?>
-<robot xmlns:xacro="http://www.ros.org/wiki/xacro">
-  <xacro:macro name="so101_gripper">
-    <!-- Gripper Base Joint -->
-    <joint name="gripper_base_joint" type="fixed">
-      <parent link="link6"/>
-      <child link="gripper_base_link"/>
-      <origin xyz="0 0 0.02" rpy="0 0 0"/>
-    </joint>
-    <!-- Gripper Base Link -->
-    <link name="gripper_base_link">
-      <visual>
-        <origin xyz="0 0 0.015" rpy="0 0 0"/>
-        <geometry>
-          <box size="0.04 0.06 0.03"/>
-        </geometry>
-        <material name="blue"/>
-      </visual>
-      <collision>
-        <origin xyz="0 0 0.015" rpy="0 0 0"/>
-        <geometry>
-          <box size="0.04 0.06 0.03"/>
-        </geometry>
-      </collision>
-      <inertial>
-        <origin xyz="0 0 0.015" rpy="0 0 0"/>
-        <mass value="0.3"/>
-        <inertia ixx="${(1/12) * 0.3 * (0.06*0.06 + 0.03*0.03)}" ixy="0.0" ixz="0.0"
-                 iyy="${(1/12) * 0.3 * (0.04*0.04 + 0.03*0.03)}" iyz="0.0"
-                 izz="${(1/12) * 0.3 * (0.04*0.04 + 0.06*0.06)}"/>
-      </inertial>
-    </link>
-    <!-- Left Finger Joint -->
-    <joint name="left_finger_joint" type="prismatic">
-      <parent link="gripper_base_link"/>
-      <child link="left_finger_link"/>
-      <origin xyz="0 0.02 0.025" rpy="0 0 0"/>
-      <axis xyz="0 -1 0"/>
-      <limit lower="0.0" upper="0.015" effort="10.0" velocity="0.1"/>
-    </joint>
-    <!-- Left Finger Link -->
-    <link name="left_finger_link">
-      <visual>
-        <origin xyz="0 0 0.02" rpy="0 0 0"/>
-        <geometry>
-          <box size="0.03 0.01 0.04"/>
-        </geometry>
-        <material name="silver"/>
-      </visual>
-      <collision>
-        <origin xyz="0 0 0.02" rpy="0 0 0"/>
-        <geometry>
-          <box size="0.03 0.01 0.04"/>
-        </geometry>
-      </collision>
-      <inertial>
-        <origin xyz="0 0 0.02" rpy="0 0 0"/>
-        <mass value="0.05"/>
-        <inertia ixx="${(1/12) * 0.05 * (0.01*0.01 + 0.04*0.04)}" ixy="0.0" ixz="0.0"
-                 iyy="${(1/12) * 0.05 * (0.03*0.03 + 0.04*0.04)}" iyz="0.0"
-                 izz="${(1/12) * 0.05 * (0.03*0.03 + 0.01*0.01)}"/>
-      </inertial>
-    </link>
-    <!-- Right Finger Joint -->
-    <joint name="right_finger_joint" type="prismatic">
-      <parent link="gripper_base_link"/>
-      <child link="right_finger_link"/>
-      <origin xyz="0 -0.02 0.025" rpy="0 0 0"/>
-      <axis xyz="0 1 0"/>
-      <limit lower="0.0" upper="0.015" effort="10.0" velocity="0.1"/>
-    </joint>
-    <!-- Right Finger Link -->
-    <link name="right_finger_link">
-      <visual>
-        <origin xyz="0 0 0.02" rpy="0 0 0"/>
-        <geometry>
-          <box size="0.03 0.01 0.04"/>
-        </geometry>
-        <material name="silver"/>
-      </visual>
-      <collision>
-        <origin xyz="0 0 0.02" rpy="0 0 0"/>
-        <geometry>
-          <box size="0.03 0.01 0.04"/>
-        </geometry>
-      </collision>
-      <inertial>
-        <origin xyz="0 0 0.02" rpy="0 0 0"/>
-        <mass value="0.05"/>
-        <inertia ixx="${(1/12) * 0.05 * (0.01*0.01 + 0.04*0.04)}" ixy="0.0" ixz="0.0"
-                 iyy="${(1/12) * 0.05 * (0.03*0.03 + 0.04*0.04)}" iyz="0.0"
-                 izz="${(1/12) * 0.05 * (0.03*0.03 + 0.01*0.01)}"/>
-      </inertial>
-    </link>
-    <!-- Self collision settings for gripper -->
-    <gazebo reference="gripper_base_link">
-      <self_collision>true</self_collision>
-    </gazebo>
-  </xacro:macro>
-</robot>
+/home/pakku/auto-trash-navigator/src/amr_description/urdf/gripper.xacro

File: install/amr_description/share/amr_description/urdf/so101_arm.xacro (robot description, xacro)
@@ -1,223 +1 @@
-<?xml version="1.0"?>
-<robot xmlns:xacro="http://www.ros.org/wiki/xacro">
-  <xacro:macro name="so101_arm">
-    <!-- Joint 1 -->
-    <joint name="joint1" type="revolute">
-      <parent link="arm_base_link"/>
-      <child link="link1"/>
-      <origin xyz="0 0 0.02" rpy="0 0 0"/>
-      <axis xyz="0 0 1"/>
-      <limit lower="-2.0" upper="2.0" effort="10.0" velocity="2.0"/>
-    </joint>
-    <!-- Link 1 -->
-    <link name="link1">
-      <visual>
-        <origin xyz="0 0 0.025" rpy="0 0 0"/>
-        <geometry>
-          <cylinder radius="0.03" length="0.05"/>
-        </geometry>
-        <material name="silver"/>
-      </visual>
-      <collision>
-        <origin xyz="0 0 0.025" rpy="0 0 0"/>
-        <geometry>
-          <cylinder radius="0.03" length="0.05"/>
-        </geometry>
-      </collision>
-      <inertial>
-        <origin xyz="0 0 0.025" rpy="0 0 0"/>
-        <mass value="0.2"/>
-        <inertia ixx="${(1/12) * 0.2 * (3*0.03*0.03 + 0.05*0.05)}" ixy="0.0" ixz="0.0"
-                 iyy="${(1/12) * 0.2 * (3*0.03*0.03 + 0.05*0.05)}" iyz="0.0"
-                 izz="${0.5 * 0.2 * 0.03 * 0.03}"/>
-      </inertial>
-    </link>
-    <!-- Joint 2 -->
-    <joint name="joint2" type="revolute">
-      <parent link="link1"/>
-      <child link="link2"/>
-      <origin xyz="0 0 0.05" rpy="0 0 0"/>
-      <axis xyz="0 1 0"/>
-      <limit lower="-2.0" upper="2.0" effort="10.0" velocity="2.0"/>
-    </joint>
-    <!-- Link 2 -->
-    <link name="link2">
-      <visual>
-        <origin xyz="0 0 0.075" rpy="0 0 0"/>
-        <geometry>
-          <box size="0.04 0.04 0.15"/>
-        </geometry>
-        <material name="blue"/>
-      </visual>
-      <collision>
-        <origin xyz="0 0 0.075" rpy="0 0 0"/>
-        <geometry>
-          <box size="0.04 0.04 0.15"/>
-        </geometry>
-      </collision>
-      <inertial>
-        <origin xyz="0 0 0.075" rpy="0 0 0"/>
-        <mass value="0.4"/>
-        <inertia ixx="${(1/12) * 0.4 * (0.04*0.04 + 0.15*0.15)}" ixy="0.0" ixz="0.0"
-                 iyy="${(1/12) * 0.4 * (0.04*0.04 + 0.15*0.15)}" iyz="0.0"
-                 izz="${(1/12) * 0.4 * (0.04*0.04 + 0.04*0.04)}"/>
-      </inertial>
-    </link>
-    <!-- Joint 3 -->
-    <joint name="joint3" type="revolute">
-      <parent link="link2"/>
-      <child link="link3"/>
-      <origin xyz="0 0 0.15" rpy="0 0 0"/>
-      <axis xyz="0 1 0"/>
-      <limit lower="-2.0" upper="2.0" effort="10.0" velocity="2.0"/>
-    </joint>
-    <!-- Link 3 -->
-    <link name="link3">
-      <visual>
-        <origin xyz="0 0 0.075" rpy="0 0 0"/>
-        <geometry>
-          <box size="0.03 0.03 0.15"/>
-        </geometry>
-        <material name="silver"/>
-      </visual>
-      <collision>
-        <origin xyz="0 0 0.075" rpy="0 0 0"/>
-        <geometry>
-          <box size="0.03 0.03 0.15"/>
-        </geometry>
-      </collision>
-      <inertial>
-        <origin xyz="0 0 0.075" rpy="0 0 0"/>
-        <mass value="0.3"/>
-        <inertia ixx="${(1/12) * 0.3 * (0.03*0.03 + 0.15*0.15)}" ixy="0.0" ixz="0.0"
-                 iyy="${(1/12) * 0.3 * (0.03*0.03 + 0.15*0.15)}" iyz="0.0"
-                 izz="${(1/12) * 0.3 * (0.03*0.03 + 0.03*0.03)}"/>
-      </inertial>
-    </link>
-    <!-- Joint 4 -->
-    <joint name="joint4" type="revolute">
-      <parent link="link3"/>
-      <child link="link4"/>
-      <origin xyz="0 0 0.15" rpy="0 0 0"/>
-      <axis xyz="0 0 1"/>
-      <limit lower="-2.0" upper="2.0" effort="10.0" velocity="2.0"/>
-    </joint>
-    <!-- Link 4 -->
-    <link name="link4">
-      <visual>
-        <origin xyz="0 0 0.02" rpy="0 0 0"/>
-        <geometry>
-          <cylinder radius="0.02" length="0.04"/>
-        </geometry>
-        <material name="blue"/>
-      </visual>
-      <collision>
-        <origin xyz="0 0 0.02" rpy="0 0 0"/>
-        <geometry>
-          <cylinder radius="0.02" length="0.04"/>
-        </geometry>
-      </collision>
-      <inertial>
-        <origin xyz="0 0 0.02" rpy="0 0 0"/>
-        <mass value="0.15"/>
-        <inertia ixx="${(1/12) * 0.15 * (3*0.02*0.02 + 0.04*0.04)}" ixy="0.0" ixz="0.0"
-                 iyy="${(1/12) * 0.15 * (3*0.02*0.02 + 0.04*0.04)}" iyz="0.0"
-                 izz="${0.5 * 0.15 * 0.02 * 0.02}"/>
-      </inertial>
-    </link>
-    <!-- Joint 5 -->
-    <joint name="joint5" type="revolute">
-      <parent link="link4"/>
-      <child link="link5"/>
-      <origin xyz="0 0 0.04" rpy="0 0 0"/>
-      <axis xyz="0 1 0"/>
-      <limit lower="-2.0" upper="2.0" effort="10.0" velocity="2.0"/>
-    </joint>
-    <!-- Link 5 -->
-    <link name="link5">
-      <visual>
-        <origin xyz="0 0 0.02" rpy="0 0 0"/>
-        <geometry>
-          <box size="0.03 0.04 0.04"/>
-        </geometry>
-        <material name="silver"/>
-      </visual>
-      <collision>
-        <origin xyz="0 0 0.02" rpy="0 0 0"/>
-        <geometry>
-          <box size="0.03 0.04 0.04"/>
-        </geometry>
-      </collision>
-      <inertial>
-        <origin xyz="0 0 0.02" rpy="0 0 0"/>
-        <mass value="0.15"/>
-        <inertia ixx="${(1/12) * 0.15 * (0.04*0.04 + 0.04*0.04)}" ixy="0.0" ixz="0.0"
-                 iyy="${(1/12) * 0.15 * (0.03*0.03 + 0.04*0.04)}" iyz="0.0"
-                 izz="${(1/12) * 0.15 * (0.03*0.03 + 0.04*0.04)}"/>
-      </inertial>
-    </link>
-    <!-- Joint 6 -->
-    <joint name="joint6" type="revolute">
-      <parent link="link5"/>
-      <child link="link6"/>
-      <origin xyz="0 0 0.04" rpy="0 0 0"/>
-      <axis xyz="0 0 1"/>
-      <limit lower="-2.0" upper="2.0" effort="10.0" velocity="2.0"/>
-    </joint>
-    <!-- Link 6 -->
-    <link name="link6">
-      <visual>
-        <origin xyz="0 0 0.01" rpy="0 0 0"/>
-        <geometry>
-          <cylinder radius="0.02" length="0.02"/>
-        </geometry>
-        <material name="blue"/>
-      </visual>
-      <collision>
-        <origin xyz="0 0 0.01" rpy="0 0 0"/>
-        <geometry>
-          <cylinder radius="0.02" length="0.02"/>
-        </geometry>
-      </collision>
-      <inertial>
-        <origin xyz="0 0 0.01" rpy="0 0 0"/>
-        <mass value="0.15"/>
-        <inertia ixx="${(1/12) * 0.15 * (3*0.02*0.02 + 0.02*0.02)}" ixy="0.0" ixz="0.0"
-                 iyy="${(1/12) * 0.15 * (3*0.02*0.02 + 0.02*0.02)}" iyz="0.0"
-                 izz="${0.5 * 0.15 * 0.02 * 0.02}"/>
-      </inertial>
-    </link>
-    <!-- Wrist Camera Joint -->
-    <joint name="wrist_camera_joint" type="fixed">
-      <parent link="link6"/>
-      <child link="wrist_camera_link"/>
-      <origin xyz="0 0.02 0.02" rpy="0 0 0"/>
-    </joint>
-    <!-- Wrist Camera Link -->
-    <link name="wrist_camera_link">
-      <visual>
-        <origin xyz="0 0 0" rpy="0 0 0"/>
-        <geometry>
-          <box size="0.01 0.02 0.01"/>
-        </geometry>
-        <material name="black"/>
-      </visual>
-      <collision>
-        <origin xyz="0 0 0" rpy="0 0 0"/>
-        <geometry>
-          <box size="0.01 0.02 0.01"/>
-        </geometry>
-      </collision>
-    </link>
-    <!-- Self collision settings for arm links -->
-    <gazebo reference="link1">
-      <self_collision>true</self_collision>
-    </gazebo>
-    <gazebo reference="link2">
-      <self_collision>true</self_collision>
-    </gazebo>
-    <gazebo reference="link3">
-      <self_collision>true</self_collision>
-    </gazebo>
-  </xacro:macro>
-</robot>
+/home/pakku/auto-trash-navigator/src/amr_description/urdf/so101_arm.xacro
