Commit message: Phase 2-C: slam_toolbox + my_map

File: src/amr_description/urdf/amr_robot.urdf.xacro (robot description, xacro)
@@ -45,4 +45,31 @@
                iyy="${(1/12) * 0.15 * (0.03*0.03 + 0.03*0.03)}" iyz="0.0"
                izz="${(1/12) * 0.15 * (0.03*0.03 + 0.1*0.1)}"/>
+    </inertial>
+  </link>
+  <joint name="lidar_joint" type="fixed">
+    <parent link="base_link"/>
+    <child link="lidar_link"/>
+    <origin xyz="-0.05 0 0.125" rpy="0 0 0"/>
+  </joint>
+  <link name="lidar_link">
+    <visual>
+      <origin xyz="0 0 0" rpy="0 0 0"/>
+      <geometry>
+        <cylinder radius="0.03" length="0.03"/>
+      </geometry>
+      <material name="black"/>
+    </visual>
+    <collision>
+      <origin xyz="0 0 0" rpy="0 0 0"/>
+      <geometry>
+        <cylinder radius="0.03" length="0.03"/>
+      </geometry>
+    </collision>
+    <inertial>
+      <origin xyz="0 0 0" rpy="0 0 0"/>
+      <mass value="0.1"/>
+      <inertia ixx="${(1/12) * 0.1 * (3*0.03*0.03 + 0.03*0.03)}" ixy="0.0" ixz="0.0"
+               iyy="${(1/12) * 0.1 * (3*0.03*0.03 + 0.03*0.03)}" iyz="0.0"
+               izz="${0.5 * 0.1 * 0.03 * 0.03}"/>
     </inertial>
   </link>
@@ -175,4 +202,28 @@
     </sensor>
   </gazebo>
+  <!-- 360 Degree 2D LiDAR Sensor -->
+  <gazebo reference="lidar_link">
+    <sensor name="gpu_lidar" type="gpu_lidar">
+      <always_on>1</always_on>
+      <update_rate>10</update_rate>
+      <visualize>true</visualize>
+      <topic>/lidar</topic>
+      <lidar>
+        <scan>
+          <horizontal>
+            <samples>360</samples>
+            <resolution>1</resolution>
+            <min_angle>-3.14159</min_angle>
+            <max_angle>3.14159</max_angle>
+          </horizontal>
+        </scan>
+        <range>
+          <min>0.15</min>
+          <max>12.0</max>
+        </range>
+      </lidar>
+      <gz_frame_id>lidar_link</gz_frame_id>
+    </sensor>
+  </gazebo>
   <!-- Gazebo Sim Sensor Plugins -->
   <gazebo>
