Commit message: fix: invert wheel joint axis polarity (all-axis drive inversion, diag 2)
Co-Authored-By: Claude Fable 5 <noreply@anthropic.com>

File: src/amr_description/urdf/base_omni_4wheel.xacro (robot description, xacro)
@@ -7,5 +7,5 @@
       <child link="${prefix}_wheel_link"/>
       <origin xyz="${x_reflect * 0.15} ${y_reflect * 0.18} -0.05" rpy="0 0 0"/>
-      <axis xyz="0 -1 0"/>
+      <axis xyz="0 1 0"/>
       <limit effort="100.0" velocity="20.0"/>
     </joint>
