Commit message: fix: correct joint2/3/5 effort limits (URDF model correction, human-approved)
loop3 root-caused the "arm never returns home after Grasp" bug to
joint2's effort limit (0.6 N*m) being physically insufficient: at
Grasp pitch=60deg, joint2 sits within ~0.001-0.025rad of its 1.65rad
hard limit for every reachable point (confirmed by an IK sweep across
the whole reachable region), and the gravity torque there was computed
from CAD (598g mass beyond J2, 226mm combined moment arm) at ~1.32N*m
-- 2.2x the old effort limit. This is a URDF modeling error, not a
motion-range change: STS3215's actual stall torque is 1.9N*m.

Corrected joint2/joint3 (pitch axes carrying the most gravity load) to
1.5N*m (1.14x the computed 1.32N*m requirement, 79% of stall) and
joint5 (wrist pitch, lighter distal load) to 0.9N*m. joint1/4/6 (yaw
axes, minimal gravity moment) stay at 0.6N*m. Verified via direct
/joint_states measurement: after this fix, a Grasp-then-home cycle at
the same point that previously pinned joint2 at exactly 1.65rad now
returns joint2 to ~-0.006rad on the first attempt, no retries needed.

Also, since amr_controllers.yaml's arm_controller previously had no
goal/path tolerance constraints (reported SUCCEEDED regardless of
actual arrival -- the reason loop3's stuck-arm bug went undetected for
so long), added explicit goal tolerance (0.08rad, trajectory tolerance
disabled since path-following lag is normal mid-motion) and made
send_arm_trajectory check the actual FollowJointTrajectory error_code
instead of just "did a result arrive".

pick_and_place.py also gained (a) solve_ik(seed_home=...) and
avoid_collisions=... options -- tried enabling both for the grasp
search but reverted (each made the IK search dramatically slower,
sometimes not converging within 90s), keeping only avoid_collisions/
seed_home=False as before; (b) find_grasp_target() now computes
joint_margin() (distance from joint limits) for logging/diagnostics
and could prefer larger-margin candidates via candidate_cap, but this
is left at 1 (first solvable candidate wins) for speed -- the effort
fix is what actually resolves the stuck-joint issue, not solution
selection.

Co-Authored-By: Claude Sonnet 5 <noreply@anthropic.com>

File: src/amr_description/urdf/so101_arm.xacro (robot description, xacro)
@@ -43,4 +43,13 @@
     </link>
     <!-- ===== Joint 2 : 肩ピッチ (X) ===== -->
+    <!-- 2026-08-10: effortをモデル訂正。CAD実測に基づき、J2より先の
+         質量598g・合成重心距離226mmから、腕が水平になる最悪ケースの
+         重力トルクは 0.598kg * 9.81 * 0.226m ≈ 1.32 N・m と算出される。
+         旧値 effort=0.6 はこれの45%しかなく自重すら支えられない
+         (実際にGrasp姿勢近傍でjoint2が可動域限界に物理的に固着し、
+         二度と戻れなくなる不具合の直接原因と特定済み)。
+         実機サーボ STS3215 のストールトルクは1.9N・mであり、
+         1.5N・m(必要1.32N・mの1.14倍、ストールの79%)は実機でも
+         成立する範囲としてeffortを訂正する。 -->
     <joint name="joint2" type="revolute">
       <parent link="link1"/>
@@ -48,5 +57,5 @@
       <origin xyz="0 0 0.06445" rpy="0 0 0"/>
       <axis xyz="1 0 0"/>
-      <limit lower="-1.65" upper="1.65" effort="0.6" velocity="2.2"/>
+      <limit lower="-1.65" upper="1.65" effort="1.5" velocity="2.2"/>
       <dynamics damping="1.0" friction="0.4"/>
     </joint>
@@ -70,4 +79,8 @@
     </link>
     <!-- ===== Joint 3 : 肘ピッチ (X) ===== -->
+    <!-- 2026-08-10: joint2と同じ理由でeffortをモデル訂正(重力
+         モーメントを受けるピッチ軸)。J3より先の質量はJ2より先より
+         小さいが、同じくSTS3215サーボ(ストール1.9N・m)を想定し、
+         安全側にjoint2と同じ1.5N・mへ引き上げる。 -->
     <joint name="joint3" type="revolute">
       <parent link="link2"/>
@@ -75,5 +88,5 @@
       <origin xyz="0 0 0.10000" rpy="0 0 0"/>
       <axis xyz="1 0 0"/>
-      <limit lower="-1.66" upper="1.66" effort="0.6" velocity="2.2"/>
+      <limit lower="-1.66" upper="1.66" effort="1.5" velocity="2.2"/>
       <dynamics damping="0.8" friction="0.3"/>
     </joint>
@@ -124,4 +137,8 @@
     </link>
     <!-- ===== Joint 5 : 手首ピッチ (X) ===== -->
+    <!-- 2026-08-10: effortをモデル訂正。手首ピッチは先端側(link5,
+         link6,グリッパー)のみを支えるため質量負荷はjoint2/3より
+         小さいが、同様に重力モーメントを受けるピッチ軸であるため
+         0.6 → 0.9 N・m(STS3215ストール1.9N・mの47%)へ引き上げる。 -->
     <joint name="joint5" type="revolute">
       <parent link="link4"/>
@@ -129,5 +146,5 @@
       <origin xyz="0 0 0.04245" rpy="0 0 0"/>
       <axis xyz="1 0 0"/>
-      <limit lower="-1.66" upper="1.66" effort="0.6" velocity="2.2"/>
+      <limit lower="-1.66" upper="1.66" effort="0.9" velocity="2.2"/>
       <dynamics damping="0.5" friction="0.2"/>
     </joint>
