Commit message: Phase 3: Add paper trash models and implement trash detector node

File: src/amr_description/urdf/amr_robot.urdf.xacro (robot description, xacro)
@@ -47,4 +47,10 @@
     </inertial>
   </link>
+  <joint name="oak_d_optical_joint" type="fixed">
+    <parent link="oak_d_link"/>
+    <child link="oak_d_optical_link"/>
+    <origin xyz="0 0 0" rpy="-1.5707963 0 -1.5707963"/>
+  </joint>
+  <link name="oak_d_optical_link"/>
   <joint name="lidar_joint" type="fixed">
     <parent link="base_link"/>

Commit message: checkpoint before local-LLM edits

File: src/amr_description/urdf/amr_robot.urdf.xacro (robot description, xacro)
@@ -108,23 +108,4 @@
     <self_collision>false</self_collision>
   </gazebo>
-  <!-- Explicitly disable collisions between wheels and base_link to prevent physics lockup -->
-  <gazebo>
-    <disable_collisions>
-      <link1>base_link</link1>
-      <link2>front_left_wheel_link</link2>
-    </disable_collisions>
-    <disable_collisions>
-      <link1>base_link</link1>
-      <link2>front_right_wheel_link</link2>
-    </disable_collisions>
-    <disable_collisions>
-      <link1>base_link</link1>
-      <link2>rear_left_wheel_link</link2>
-    </disable_collisions>
-    <disable_collisions>
-      <link1>base_link</link1>
-      <link2>rear_right_wheel_link</link2>
-    </disable_collisions>
-  </gazebo>
   <!-- ros2_control configuration for arm and gripper -->
   <ros2_control name="amr_robot_system" type="system">
@@ -195,5 +176,6 @@
     <plugin filename="gz_ros2_control-system" name="gz_ros2_control::GazeboSimROS2ControlPlugin">
       <parameters>$(find amr_description)/config/amr_controllers.yaml</parameters>
-      <hold_joints>true</hold_joints>
+      <hold_joints>false</hold_joints>
+      <position_proportional_gain>1000.0</position_proportional_gain>
     </plugin>
   </gazebo>

File: src/amr_description/urdf/base_omni_4wheel.xacro (robot description, xacro)
@@ -6,6 +6,7 @@
       <parent link="base_link"/>
       <child link="${prefix}_wheel_link"/>
-      <origin xyz="${x_reflect * 0.15} ${y_reflect * 0.18} -0.05" rpy="0 0 ${(1 - y_reflect) * pi / 2}"/>
-      <axis xyz="0 ${y_reflect} 0"/>
+      <origin xyz="${x_reflect * 0.15} ${y_reflect * 0.18} -0.05" rpy="0 0 0"/>
+      <axis xyz="0 -1 0"/>
+      <limit effort="100.0" velocity="20.0"/>
     </joint>
     <link name="${prefix}_wheel_link">
@@ -32,4 +33,5 @@
     </link>
     <gazebo reference="${prefix}_wheel_link">
+      <self_collision>false</self_collision>
       <collision name="${prefix}_wheel_link_collision">
         <surface>
@@ -54,7 +56,7 @@
   <xacro:macro name="base_omni_4wheel">
     <xacro:omni_wheel prefix="front_left" x_reflect="1" y_reflect="1" fdir="1 -1 0"/>
-    <xacro:omni_wheel prefix="front_right" x_reflect="1" y_reflect="-1" fdir="1 1 0"/>
+    <xacro:omni_wheel prefix="front_right" x_reflect="1" y_reflect="-1" fdir="-1 -1 0"/>
     <xacro:omni_wheel prefix="rear_left" x_reflect="-1" y_reflect="1" fdir="1 1 0"/>
-    <xacro:omni_wheel prefix="rear_right" x_reflect="-1" y_reflect="-1" fdir="1 -1 0"/>
+    <xacro:omni_wheel prefix="rear_right" x_reflect="-1" y_reflect="-1" fdir="-1 1 0"/>
     <!-- Mecanum Drive Plugin for Gazebo Sim -->
     <gazebo>

File: src/amr_description/urdf/gripper.xacro (robot description, xacro)
@@ -95,5 +95,5 @@
     <!-- Self collision settings for gripper -->
     <gazebo reference="gripper_base_link">
-      <self_collision>true</self_collision>
+      <self_collision>false</self_collision>
     </gazebo>
   </xacro:macro>

File: src/amr_description/urdf/so101_arm.xacro (robot description, xacro)
@@ -9,4 +9,5 @@
       <axis xyz="0 0 1"/>
       <limit lower="-2.0" upper="2.0" effort="10.0" velocity="2.0"/>
+      <dynamics damping="10.0" friction="5.0"/>
     </joint>
     <!-- Link 1 -->
@@ -40,4 +41,5 @@
       <axis xyz="0 1 0"/>
       <limit lower="-2.0" upper="2.0" effort="10.0" velocity="2.0"/>
+      <dynamics damping="30.0" friction="25.0"/>
     </joint>
     <!-- Link 2 -->
@@ -71,4 +73,5 @@
       <axis xyz="0 1 0"/>
       <limit lower="-2.0" upper="2.0" effort="10.0" velocity="2.0"/>
+      <dynamics damping="20.0" friction="15.0"/>
     </joint>
     <!-- Link 3 -->
@@ -102,4 +105,5 @@
       <axis xyz="0 0 1"/>
       <limit lower="-2.0" upper="2.0" effort="10.0" velocity="2.0"/>
+      <dynamics damping="10.0" friction="5.0"/>
     </joint>
     <!-- Link 4 -->
@@ -133,4 +137,5 @@
       <axis xyz="0 1 0"/>
       <limit lower="-2.0" upper="2.0" effort="10.0" velocity="2.0"/>
+      <dynamics damping="20.0" friction="15.0"/>
     </joint>
     <!-- Link 5 -->
@@ -164,4 +169,5 @@
       <axis xyz="0 0 1"/>
       <limit lower="-2.0" upper="2.0" effort="10.0" velocity="2.0"/>
+      <dynamics damping="10.0" friction="5.0"/>
     </joint>
     <!-- Link 6 -->
@@ -212,11 +218,11 @@
     <!-- Self collision settings for arm links -->
     <gazebo reference="link1">
-      <self_collision>true</self_collision>
+      <self_collision>false</self_collision>
     </gazebo>
     <gazebo reference="link2">
-      <self_collision>true</self_collision>
+      <self_collision>false</self_collision>
     </gazebo>
     <gazebo reference="link3">
-      <self_collision>true</self_collision>
+      <self_collision>false</self_collision>
     </gazebo>
   </xacro:macro>

Commit message: wip: chassis geometry for real hardware (base_link height, wheels)

File: src/amr_description/urdf/amr_robot.urdf.xacro (robot description, xacro)
@@ -5,22 +5,33 @@
   <material name="black"><color rgba="0.1 0.1 0.1 1.0"/></material>
   <link name="base_footprint"/>
+  <!-- 2026-08-24 実機HW確定(feature/hw-v2): base_link原点高さ(z)の算出根拠。
+       確定仕様(base_footprint基準): 車輪半径0.040 / 主板上面z=0.060。
+       base_linkを主板の板厚を表す薄い箱とし、下面=車輪中心高さ(接地条件、
+       車輪半径と一致=0.040)、上面=主板上面(0.060)となるように定義する。
+         板厚 = 0.060 - 0.040 = 0.020
+         base_link原点(中心)z = (0.040 + 0.060) / 2 = 0.050
+       この結果、子リンク(車輪, arm_base, oak_d, lidar)のjoint origin zは
+       「絶対値(base_footprint基準) - 0.050」で算出する。
+       検算: 旧値(base_link z=0.1, 板厚0.15)は 底面=0.025 上面=0.175 で
+       あり、旧arm_base_joint z=0.075→arm_base_link絶対z=0.175。
+       新: 底面=0.040(旧0.025から車輪半径分上昇)上面=0.060。 -->
   <joint name="base_joint" type="fixed">
     <parent link="base_footprint"/>
     <child link="base_link"/>
-    <origin xyz="0 0 0.1" rpy="0 0 0"/>
+    <origin xyz="0 0 0.050" rpy="0 0 0"/>
   </joint>
   <link name="base_link">
     <visual>
-      <geometry><box size="0.4 0.4 0.15"/></geometry>
+      <geometry><box size="0.4 0.4 0.02"/></geometry>
       <material name="silver"/>
     </visual>
     <collision>
-      <geometry><box size="0.4 0.4 0.15"/></geometry>
+      <geometry><box size="0.4 0.4 0.02"/></geometry>
     </collision>
     <inertial>
       <origin xyz="0 0 0" rpy="0 0 0"/>
       <mass value="10.0"/>
-      <inertia ixx="${(1/12) * 10.0 * (0.4*0.4 + 0.15*0.15)}" ixy="0.0" ixz="0.0"
-               iyy="${(1/12) * 10.0 * (0.4*0.4 + 0.15*0.15)}" iyz="0.0"
+      <inertia ixx="${(1/12) * 10.0 * (0.4*0.4 + 0.02*0.02)}" ixy="0.0" ixz="0.0"
+               iyy="${(1/12) * 10.0 * (0.4*0.4 + 0.02*0.02)}" iyz="0.0"
                izz="${(1/12) * 10.0 * (0.4*0.4 + 0.4*0.4)}"/>
     </inertial>
@@ -29,8 +40,13 @@
   <xacro:include filename="base_omni_4wheel.xacro"/>
   <xacro:base_omni_4wheel/>
+  <!-- 2026-08-24 実機HW確定: OAK-D Lite 光学中心 (0.182, 0.135, 0.197)
+       [base_footprint基準]、俯角25°。oak_d_optical_joint(下記、Z前方の
+       光学フレーム規約)は並進0のため、oak_d_link原点=光学中心の絶対位置
+       をそのままbase_link基準に変換すればよい: z = 0.197 - 0.050 = 0.147。
+       pitch = 25° = 0.4363323 rad(既存符号規約=正のpitchで下向きを踏襲)。 -->
   <joint name="oak_d_joint" type="fixed">
     <parent link="base_link"/>
     <child link="oak_d_link"/>
-    <origin xyz="0.18 0 0.1" rpy="0 0.26 0"/>
+    <origin xyz="0.182 0.135 0.147" rpy="0 0.4363323 0"/>
   </joint>
   <link name="oak_d_link">
@@ -53,8 +69,13 @@
   </joint>
   <link name="oak_d_optical_link"/>
+  <!-- 2026-08-24 実機HW確定: RPLIDAR A1M8。スキャン面z=0.210、
+       位置x=-0.160,y=+0.013 [base_footprint基準] → base_link基準は
+       z=0.210-0.050=0.160。取付都合で本体を90°回しているため
+       laser_frameにyaw+90°を付与(除去角度セクターの算出根拠は
+       lidar_filter.pyのコメント参照)。 -->
   <joint name="lidar_joint" type="fixed">
     <parent link="base_link"/>
     <child link="lidar_link"/>
-    <origin xyz="-0.05 0 0.125" rpy="0 0 0"/>
+    <origin xyz="-0.160 0.013 0.160" rpy="0 0 1.5707963"/>
   </joint>
   <link name="lidar_link">
@@ -80,8 +101,12 @@
     </inertial>
   </link>
+  <!-- 2026-08-24 実機HW確定: アーム取付 x=0.150,y=0,z=主板上面(0.060)
+       [base_footprint基準、Ø100フランジ] → base_link基準は
+       z=0.060-0.050=0.010。向き(rpy)は現状維持(J2正転で車体前方=+X
+       へ倒れる設計を保つためyaw+90°のまま)。 -->
   <joint name="arm_base_joint" type="fixed">
     <parent link="base_link"/>
     <child link="arm_base_link"/>
-    <origin xyz="0.15 0 0.075" rpy="0 0 1.5707963"/>
+    <origin xyz="0.150 0 0.010" rpy="0 0 1.5707963"/>
   </joint>
   <link name="arm_base_link">
@@ -228,5 +253,8 @@
         </scan>
         <range>
-          <!-- 0.45: arm sweeps within 0.45m of lidar during pick; exclude self-hits --><min>0.45</min>
+          <!-- 2026-08-24: 実機HW確定でLiDAR-アーム基部間距離が0.31m(伸展時0.51m)に
+               広がり、min rangeだけではアーム除去に不十分(伸ばしたアームがrange外に
+               出てしまう)。センサー側のminは仕様値0.15のみとし、アーム自己ヒットの
+               除去はlidar_filter.pyの角度セクターフィルタで行う。 --><min>0.15</min>
           <max>12.0</max>
         </range>

File: src/amr_description/urdf/base_omni_4wheel.xacro (robot description, xacro)
@@ -2,11 +2,18 @@
 <robot xmlns:xacro="http://www.ros.org/wiki/xacro" xmlns:gz="http://gazebosim.org/schema">
   <!-- Macro for a single omni wheel -->
+  <!-- 2026-08-24 実機HW確定(feature/hw-v2): wheel Ø80mm(半径0.040)、
+       ホイールベース240mm/トレッド360mm → 車輪位置 x=±0.120, y=±0.180。
+       z=-0.010 は base_link 原点(z=0.050, base_footprint基準)から
+       車輪中心(=車輪半径0.040, 接地条件)までのオフセット
+       (0.040 - 0.050 = -0.010)。base_linkのz算出根拠は
+       amr_robot.urdf.xacro の base_joint コメント参照。
+       joint速度上限 16.0 rad/s は 最高速度0.64m/s ÷ 半径0.040 = 16.0 -->
   <xacro:macro name="omni_wheel" params="prefix x_reflect y_reflect fdir">
     <joint name="${prefix}_wheel_joint" type="continuous">
       <parent link="base_link"/>
       <child link="${prefix}_wheel_link"/>
-      <origin xyz="${x_reflect * 0.15} ${y_reflect * 0.18} -0.05" rpy="0 0 0"/>
+      <origin xyz="${x_reflect * 0.120} ${y_reflect * 0.180} -0.010" rpy="0 0 0"/>
       <axis xyz="0 1 0"/>
-      <limit effort="100.0" velocity="20.0"/>
+      <limit effort="100.0" velocity="16.0"/>
     </joint>
     <link name="${prefix}_wheel_link">
@@ -14,5 +21,5 @@
         <origin xyz="0 0 0" rpy="${pi/2} 0 0"/>
         <geometry>
-          <cylinder radius="0.05" length="0.04"/>
+          <cylinder radius="0.040" length="0.04"/>
         </geometry>
         <material name="black"/>
@@ -21,5 +28,5 @@
         <origin xyz="0 0 0" rpy="0 0 0"/>
         <geometry>
-          <sphere radius="0.05"/>
+          <sphere radius="0.040"/>
         </geometry>
       </collision>
@@ -27,7 +34,7 @@
         <origin xyz="0 0 0" rpy="${pi/2} 0 0"/>
         <mass value="0.2"/>
-        <inertia ixx="${(1/12) * 0.2 * (3 * 0.05 * 0.05 + 0.04 * 0.04)}" ixy="0.0" ixz="0.0"
-                 iyy="${(1/12) * 0.2 * (3 * 0.05 * 0.05 + 0.04 * 0.04)}" iyz="0.0"
-                 izz="${0.5 * 0.2 * 0.05 * 0.05}"/>
+        <inertia ixx="${(1/12) * 0.2 * (3 * 0.040 * 0.040 + 0.04 * 0.04)}" ixy="0.0" ixz="0.0"
+                 iyy="${(1/12) * 0.2 * (3 * 0.040 * 0.040 + 0.04 * 0.04)}" iyz="0.0"
+                 izz="${0.5 * 0.2 * 0.040 * 0.040}"/>
       </inertial>
     </link>
@@ -68,7 +75,7 @@
         <back_left_joint>rear_left_wheel_joint</back_left_joint>
         <back_right_joint>rear_right_wheel_joint</back_right_joint>
-        <wheel_separation>0.36</wheel_separation>
-        <wheelbase>0.30</wheelbase>
-        <wheel_radius>0.05</wheel_radius>
+        <wheel_separation>0.360</wheel_separation>
+        <wheelbase>0.240</wheelbase>
+        <wheel_radius>0.040</wheel_radius>
         <topic>/cmd_vel</topic>
         <odom_topic>/odom</odom_topic>
