Commit message: feat: real CAD dimensions for SO-101 arm and gripper
Co-Authored-By: Claude Fable 5 <noreply@anthropic.com>

File: src/amr_description/urdf/amr_robot.urdf.xacro (robot description, xacro)
@@ -83,5 +83,5 @@
     <parent link="base_link"/>
     <child link="arm_base_link"/>
-    <origin xyz="0.1 0 0.075" rpy="0 0 0"/>
+    <origin xyz="0.15 0 0.075" rpy="0 0 -1.5707963"/>
   </joint>
   <link name="arm_base_link">

File: src/amr_description/urdf/gripper.xacro (robot description, xacro)
@@ -1,100 +1,105 @@
 <?xml version="1.0"?>
+<!--
+  SO-101 グリッパー — Fusion 360 実測値版 (2026-07-28)
+  機構: ラック&ピニオン 平行開閉 (モジュール2.0 / 12歯 / ピッチ半径 12.0mm)
+        2本のラックはピニオンを挟んで Y 方向に ±10.7mm オフセットし、
+        X 方向へ逆向きに動く。
+  位置 (J6原点からの +Z、CAD絶対Zから換算):
+    ピニオン軸ホーン座面 (grip基部) : 0.0534 m
+    把持面 下端                      : 0.0616 m  → gripper_base から 0.0082
+    把持面 中心 (把持点)             : 0.0741 m  → gripper_base から 0.0207
+    指先端 (TCP)                     : 0.0865 m  → gripper_base から 0.0331
+  開口: travel=0 が機構の中央で 34.0mm (把持面 x = ±17.0mm)
+        opening[mm] = 34 + 24 * theta[rad] (theta はサーボ角)
+        噛み合いを1ピッチ以上残す条件で片側 ±13mm → 開口 8mm 〜 60mm
+        よって prismatic の可動域は -0.013 〜 +0.013 m (0 = 中央 34mm)
+  力/速度: ラック推力 = トルク / ピッチ半径 = 0.6 N·m / 0.012 m = 50 N (実用値)
+           ラック速度 = 2.2 rad/s * 0.012 m = 0.026 m/s (実用値)
+  指: 把持面 23.4(Y) x 24.9(Z) mm、ポスト厚 6.0mm、1本 6.1 g
+-->
 <robot xmlns:xacro="http://www.ros.org/wiki/xacro">
   <xacro:macro name="so101_gripper">
-    <!-- Gripper Base Joint -->
+    <!-- ===== グリッパー基部 (ピニオン軸ホーン座面) ===== -->
     <joint name="gripper_base_joint" type="fixed">
       <parent link="link6"/>
       <child link="gripper_base_link"/>
-      <origin xyz="0 0 0.02" rpy="0 0 0"/>
+      <origin xyz="0 0 0.0534" rpy="0 0 0"/>
     </joint>
-    <!-- Gripper Base Link -->
     <link name="gripper_base_link">
       <visual>
-        <origin xyz="0 0 0.015" rpy="0 0 0"/>
-        <geometry>
-          <box size="0.04 0.06 0.03"/>
-        </geometry>
+        <origin xyz="0 0 0.008" rpy="0 0 0"/>
+        <geometry><box size="0.050 0.030 0.016"/></geometry>
         <material name="blue"/>
       </visual>
       <collision>
-        <origin xyz="0 0 0.015" rpy="0 0 0"/>
-        <geometry>
-          <box size="0.04 0.06 0.03"/>
-        </geometry>
+        <origin xyz="0 0 0.008" rpy="0 0 0"/>
+        <geometry><box size="0.050 0.030 0.016"/></geometry>
       </collision>
       <inertial>
-        <origin xyz="0 0 0.015" rpy="0 0 0"/>
-        <mass value="0.3"/>
-        <inertia ixx="${(1/12) * 0.3 * (0.06*0.06 + 0.03*0.03)}" ixy="0.0" ixz="0.0"
-                 iyy="${(1/12) * 0.3 * (0.04*0.04 + 0.03*0.03)}" iyz="0.0"
-                 izz="${(1/12) * 0.3 * (0.04*0.04 + 0.06*0.06)}"/>
+        <origin xyz="0 0 0.008" rpy="0 0 0"/>
+        <mass value="0.030"/>
+        <inertia ixx="${(1/12) * 0.030 * (0.030*0.030 + 0.016*0.016)}" ixy="0.0" ixz="0.0"
+                 iyy="${(1/12) * 0.030 * (0.050*0.050 + 0.016*0.016)}" iyz="0.0"
+                 izz="${(1/12) * 0.030 * (0.050*0.050 + 0.030*0.030)}"/>
       </inertial>
     </link>
-    <!-- Left Finger Joint -->
+    <!-- ===== 左指 (X負側のラック、Y +10.7mm 側) =====
+         joint 値 0 = 把持面 x = -0.017 (開口34mm)
+         正方向 = 開く (-X へ移動) -->
     <joint name="left_finger_joint" type="prismatic">
       <parent link="gripper_base_link"/>
       <child link="left_finger_link"/>
-      <origin xyz="0 0.02 0.025" rpy="0 0 0"/>
-      <axis xyz="0 -1 0"/>
-      <limit lower="0.0" upper="0.015" effort="10.0" velocity="0.1"/>
+      <origin xyz="-0.020 0.0107 0" rpy="0 0 0"/>
+      <axis xyz="-1 0 0"/>
+      <limit lower="-0.013" upper="0.013" effort="50.0" velocity="0.026"/>
+      <dynamics damping="5.0" friction="1.0"/>
     </joint>
-    <!-- Left Finger Link -->
     <link name="left_finger_link">
       <visual>
-        <origin xyz="0 0 0.02" rpy="0 0 0"/>
-        <geometry>
-          <box size="0.03 0.01 0.04"/>
-        </geometry>
+        <origin xyz="0 0 0.0207" rpy="0 0 0"/>
+        <geometry><box size="0.006 0.0234 0.0249"/></geometry>
         <material name="silver"/>
       </visual>
       <collision>
-        <origin xyz="0 0 0.02" rpy="0 0 0"/>
-        <geometry>
-          <box size="0.03 0.01 0.04"/>
-        </geometry>
+        <origin xyz="0 0 0.0207" rpy="0 0 0"/>
+        <geometry><box size="0.006 0.0234 0.0249"/></geometry>
       </collision>
       <inertial>
-        <origin xyz="0 0 0.02" rpy="0 0 0"/>
-        <mass value="0.05"/>
-        <inertia ixx="${(1/12) * 0.05 * (0.01*0.01 + 0.04*0.04)}" ixy="0.0" ixz="0.0"
-                 iyy="${(1/12) * 0.05 * (0.03*0.03 + 0.04*0.04)}" iyz="0.0"
-                 izz="${(1/12) * 0.05 * (0.03*0.03 + 0.01*0.01)}"/>
+        <origin xyz="0.0089 0 0.0152" rpy="0 0 0"/>
+        <mass value="0.0061"/>
+        <inertia ixx="${(1/12) * 0.0061 * (0.0234*0.0234 + 0.0249*0.0249)}" ixy="0.0" ixz="0.0"
+                 iyy="${(1/12) * 0.0061 * (0.006*0.006 + 0.0249*0.0249)}" iyz="0.0"
+                 izz="${(1/12) * 0.0061 * (0.006*0.006 + 0.0234*0.0234)}"/>
       </inertial>
     </link>
-    <!-- Right Finger Joint -->
+    <!-- ===== 右指 (X正側のラック、Y -10.7mm 側) ===== -->
     <joint name="right_finger_joint" type="prismatic">
       <parent link="gripper_base_link"/>
       <child link="right_finger_link"/>
-      <origin xyz="0 -0.02 0.025" rpy="0 0 0"/>
-      <axis xyz="0 1 0"/>
-      <limit lower="0.0" upper="0.015" effort="10.0" velocity="0.1"/>
+      <origin xyz="0.020 -0.0107 0" rpy="0 0 0"/>
+      <axis xyz="1 0 0"/>
+      <limit lower="-0.013" upper="0.013" effort="50.0" velocity="0.026"/>
+      <dynamics damping="5.0" friction="1.0"/>
+      <mimic joint="left_finger_joint" multiplier="1.0" offset="0.0"/>
     </joint>
-    <!-- Right Finger Link -->
     <link name="right_finger_link">
       <visual>
-        <origin xyz="0 0 0.02" rpy="0 0 0"/>
-        <geometry>
-          <box size="0.03 0.01 0.04"/>
-        </geometry>
+        <origin xyz="0 0 0.0207" rpy="0 0 0"/>
+        <geometry><box size="0.006 0.0234 0.0249"/></geometry>
         <material name="silver"/>
       </visual>
       <collision>
-        <origin xyz="0 0 0.02" rpy="0 0 0"/>
-        <geometry>
-          <box size="0.03 0.01 0.04"/>
-        </geometry>
+        <origin xyz="0 0 0.0207" rpy="0 0 0"/>
+        <geometry><box size="0.006 0.0234 0.0249"/></geometry>
       </collision>
       <inertial>
-        <origin xyz="0 0 0.02" rpy="0 0 0"/>
-        <mass value="0.05"/>
-        <inertia ixx="${(1/12) * 0.05 * (0.01*0.01 + 0.04*0.04)}" ixy="0.0" ixz="0.0"
-                 iyy="${(1/12) * 0.05 * (0.03*0.03 + 0.04*0.04)}" iyz="0.0"
-                 izz="${(1/12) * 0.05 * (0.03*0.03 + 0.01*0.01)}"/>
+        <origin xyz="-0.0089 0 0.0152" rpy="0 0 0"/>
+        <mass value="0.0061"/>
+        <inertia ixx="${(1/12) * 0.0061 * (0.0234*0.0234 + 0.0249*0.0249)}" ixy="0.0" ixz="0.0"
+                 iyy="${(1/12) * 0.0061 * (0.006*0.006 + 0.0249*0.0249)}" iyz="0.0"
+                 izz="${(1/12) * 0.0061 * (0.006*0.006 + 0.0234*0.0234)}"/>
       </inertial>
     </link>
-    <!-- Self collision settings for gripper -->
-    <gazebo reference="gripper_base_link">
-      <self_collision>false</self_collision>
-    </gazebo>
+    <gazebo reference="gripper_base_link"><self_collision>false</self_collision></gazebo>
   </xacro:macro>
 </robot>

File: src/amr_description/urdf/so101_arm.xacro (robot description, xacro)
@@ -1,229 +1,222 @@
 <?xml version="1.0"?>
+<!--
+  SO-101 6軸アーム — Fusion 360 実測値版 (2026-07-28)
+  リンク長: 全て前ジョイントからの +Z オフセット (CAD実測、単位 m)
+    j1 0.04350 / j2 0.06445 / j3 0.10000 / j4 0.09755 / j5 0.04245 / j6 0.06855
+    grasp(把持点) 0.07410 / tcp(指先) 0.08650   ※ベース底面からの全高 0.503 m
+  回転軸: Z-X-X-Z-X-Z (j2 を正に回すとアームは +Y 方向へ倒れる / 右ねじ)
+  可動域: サーボ+ホーン+ネジ込みの実測限界から安全側に設定
+  質量・重心: PLA 1.24 g/cm3 + STS3215 55g/個 で算出した CAD 実測値
+  effort/velocity: STS3215 のストール 1.9 N·m / 無負荷 4.4 rad/s に対する実用値
+  慣性テンソル: リンク外形の円柱/直方体近似 (実測質量・重心を使用)
+  注意: ゼロ姿勢 = 全関節 0 = 6軸すべてZ軸上に一直線 (真上)。
+        実機組立後に各サーボへ Set Middle Position を打ち、機械ゼロ=2048=0rad を保証すること。
+-->
 <robot xmlns:xacro="http://www.ros.org/wiki/xacro">
   <xacro:macro name="so101_arm">
-    <!-- Joint 1 -->
+    <!-- ===== Joint 1 : ベース旋回 (Z) ===== -->
     <joint name="joint1" type="revolute">
       <parent link="arm_base_link"/>
       <child link="link1"/>
-      <origin xyz="0 0 0.02" rpy="0 0 0"/>
+      <origin xyz="0 0 0.04350" rpy="0 0 0"/>
       <axis xyz="0 0 1"/>
-      <limit lower="-2.0" upper="2.0" effort="10.0" velocity="2.0"/>
-      <dynamics damping="10.0" friction="5.0"/>
-    </joint>
-    <!-- Link 1 -->
+      <limit lower="-3.05" upper="3.05" effort="0.6" velocity="2.2"/>
+      <dynamics damping="0.5" friction="0.2"/>
+    </joint>
     <link name="link1">
       <visual>
-        <origin xyz="0 0 0.025" rpy="0 0 0"/>
-        <geometry>
-          <cylinder radius="0.03" length="0.05"/>
-        </geometry>
+        <origin xyz="0 0 0.03223" rpy="0 0 0"/>
+        <geometry><cylinder radius="0.030" length="0.06445"/></geometry>
         <material name="silver"/>
       </visual>
       <collision>
-        <origin xyz="0 0 0.025" rpy="0 0 0"/>
-        <geometry>
-          <cylinder radius="0.03" length="0.05"/>
-        </geometry>
-      </collision>
-      <inertial>
-        <origin xyz="0 0 0.025" rpy="0 0 0"/>
-        <mass value="0.2"/>
-        <inertia ixx="${(1/12) * 0.2 * (3*0.03*0.03 + 0.05*0.05)}" ixy="0.0" ixz="0.0"
-                 iyy="${(1/12) * 0.2 * (3*0.03*0.03 + 0.05*0.05)}" iyz="0.0"
-                 izz="${0.5 * 0.2 * 0.03 * 0.03}"/>
-      </inertial>
-    </link>
-    <!-- Joint 2 -->
+        <origin xyz="0 0 0.03223" rpy="0 0 0"/>
+        <geometry><cylinder radius="0.030" length="0.06445"/></geometry>
+      </collision>
+      <inertial>
+        <origin xyz="-0.0006 0 0.0339" rpy="0 0 0"/>
+        <mass value="0.1476"/>
+        <inertia ixx="${(1/12) * 0.1476 * (3*0.030*0.030 + 0.06445*0.06445)}" ixy="0.0" ixz="0.0"
+                 iyy="${(1/12) * 0.1476 * (3*0.030*0.030 + 0.06445*0.06445)}" iyz="0.0"
+                 izz="${0.5 * 0.1476 * 0.030 * 0.030}"/>
+      </inertial>
+    </link>
+    <!-- ===== Joint 2 : 肩ピッチ (X) ===== -->
     <joint name="joint2" type="revolute">
       <parent link="link1"/>
       <child link="link2"/>
-      <origin xyz="0 0 0.05" rpy="0 0 0"/>
-      <axis xyz="0 1 0"/>
-      <limit lower="-2.0" upper="2.0" effort="10.0" velocity="2.0"/>
-      <dynamics damping="30.0" friction="25.0"/>
-    </joint>
-    <!-- Link 2 -->
+      <origin xyz="0 0 0.06445" rpy="0 0 0"/>
+      <axis xyz="1 0 0"/>
+      <limit lower="-1.65" upper="1.65" effort="0.6" velocity="2.2"/>
+      <dynamics damping="1.0" friction="0.4"/>
+    </joint>
     <link name="link2">
       <visual>
-        <origin xyz="0 0 0.075" rpy="0 0 0"/>
-        <geometry>
-          <box size="0.04 0.04 0.15"/>
-        </geometry>
+        <origin xyz="0 0 0.05" rpy="0 0 0"/>
+        <geometry><box size="0.036 0.032 0.100"/></geometry>
         <material name="blue"/>
       </visual>
       <collision>
-        <origin xyz="0 0 0.075" rpy="0 0 0"/>
-        <geometry>
-          <box size="0.04 0.04 0.15"/>
-        </geometry>
-      </collision>
-      <inertial>
-        <origin xyz="0 0 0.075" rpy="0 0 0"/>
-        <mass value="0.4"/>
-        <inertia ixx="${(1/12) * 0.4 * (0.04*0.04 + 0.15*0.15)}" ixy="0.0" ixz="0.0"
-                 iyy="${(1/12) * 0.4 * (0.04*0.04 + 0.15*0.15)}" iyz="0.0"
-                 izz="${(1/12) * 0.4 * (0.04*0.04 + 0.04*0.04)}"/>
-      </inertial>
-    </link>
-    <!-- Joint 3 -->
+        <origin xyz="0 0 0.05" rpy="0 0 0"/>
+        <geometry><box size="0.036 0.032 0.100"/></geometry>
+      </collision>
+      <inertial>
+        <origin xyz="-0.0010 0 0.0666" rpy="0 0 0"/>
+        <mass value="0.1232"/>
+        <inertia ixx="${(1/12) * 0.1232 * (0.032*0.032 + 0.100*0.100)}" ixy="0.0" ixz="0.0"
+                 iyy="${(1/12) * 0.1232 * (0.036*0.036 + 0.100*0.100)}" iyz="0.0"
+                 izz="${(1/12) * 0.1232 * (0.036*0.036 + 0.032*0.032)}"/>
+      </inertial>
+    </link>
+    <!-- ===== Joint 3 : 肘ピッチ (X) ===== -->
     <joint name="joint3" type="revolute">
       <parent link="link2"/>
       <child link="link3"/>
-      <origin xyz="0 0 0.15" rpy="0 0 0"/>
-      <axis xyz="0 1 0"/>
-      <limit lower="-2.0" upper="2.0" effort="10.0" velocity="2.0"/>
-      <dynamics damping="20.0" friction="15.0"/>
-    </joint>
-    <!-- Link 3 -->
+      <origin xyz="0 0 0.10000" rpy="0 0 0"/>
+      <axis xyz="1 0 0"/>
+      <limit lower="-1.66" upper="1.66" effort="0.6" velocity="2.2"/>
+      <dynamics damping="0.8" friction="0.3"/>
+    </joint>
     <link name="link3">
       <visual>
-        <origin xyz="0 0 0.075" rpy="0 0 0"/>
-        <geometry>
-          <box size="0.03 0.03 0.15"/>
-        </geometry>
+        <origin xyz="0 0 0.04878" rpy="0 0 0"/>
+        <geometry><box size="0.032 0.028 0.09755"/></geometry>
         <material name="silver"/>
       </visual>
       <collision>
-        <origin xyz="0 0 0.075" rpy="0 0 0"/>
-        <geometry>
-          <box size="0.03 0.03 0.15"/>
-        </geometry>
-      </collision>
-      <inertial>
-        <origin xyz="0 0 0.075" rpy="0 0 0"/>
-        <mass value="0.3"/>
-        <inertia ixx="${(1/12) * 0.3 * (0.03*0.03 + 0.15*0.15)}" ixy="0.0" ixz="0.0"
-                 iyy="${(1/12) * 0.3 * (0.03*0.03 + 0.15*0.15)}" iyz="0.0"
-                 izz="${(1/12) * 0.3 * (0.03*0.03 + 0.03*0.03)}"/>
-      </inertial>
-    </link>
-    <!-- Joint 4 -->
+        <origin xyz="0 0 0.04878" rpy="0 0 0"/>
+        <geometry><box size="0.032 0.028 0.09755"/></geometry>
+      </collision>
+      <inertial>
+        <origin xyz="0.0017 0 0.0592" rpy="0 0 0"/>
+        <mass value="0.1197"/>
+        <inertia ixx="${(1/12) * 0.1197 * (0.028*0.028 + 0.09755*0.09755)}" ixy="0.0" ixz="0.0"
+                 iyy="${(1/12) * 0.1197 * (0.032*0.032 + 0.09755*0.09755)}" iyz="0.0"
+                 izz="${(1/12) * 0.1197 * (0.032*0.032 + 0.028*0.028)}"/>
+      </inertial>
+    </link>
+    <!-- ===== Joint 4 : 前腕ロール (Z) ===== -->
     <joint name="joint4" type="revolute">
       <parent link="link3"/>
       <child link="link4"/>
-      <origin xyz="0 0 0.15" rpy="0 0 0"/>
+      <origin xyz="0 0 0.09755" rpy="0 0 0"/>
       <axis xyz="0 0 1"/>
-      <limit lower="-2.0" upper="2.0" effort="10.0" velocity="2.0"/>
-      <dynamics damping="10.0" friction="5.0"/>
-    </joint>
-    <!-- Link 4 -->
+      <limit lower="-3.05" upper="3.05" effort="0.6" velocity="2.2"/>
+      <dynamics damping="0.4" friction="0.15"/>
+    </joint>
     <link name="link4">
       <visual>
-        <origin xyz="0 0 0.02" rpy="0 0 0"/>
-        <geometry>
-          <cylinder radius="0.02" length="0.04"/>
-        </geometry>
+        <origin xyz="0 0 0.02123" rpy="0 0 0"/>
+        <geometry><cylinder radius="0.022" length="0.04245"/></geometry>
         <material name="blue"/>
       </visual>
       <collision>
-        <origin xyz="0 0 0.02" rpy="0 0 0"/>
-        <geometry>
-          <cylinder radius="0.02" length="0.04"/>
-        </geometry>
-      </collision>
-      <inertial>
-        <origin xyz="0 0 0.02" rpy="0 0 0"/>
-        <mass value="0.15"/>
-        <inertia ixx="${(1/12) * 0.15 * (3*0.02*0.02 + 0.04*0.04)}" ixy="0.0" ixz="0.0"
-                 iyy="${(1/12) * 0.15 * (3*0.02*0.02 + 0.04*0.04)}" iyz="0.0"
-                 izz="${0.5 * 0.15 * 0.02 * 0.02}"/>
-      </inertial>
-    </link>
-    <!-- Joint 5 -->
+        <origin xyz="0 0 0.02123" rpy="0 0 0"/>
+        <geometry><cylinder radius="0.022" length="0.04245"/></geometry>
+      </collision>
+      <inertial>
+        <origin xyz="-0.0011 0 0.0283" rpy="0 0 0"/>
+        <mass value="0.0811"/>
+        <inertia ixx="${(1/12) * 0.0811 * (3*0.022*0.022 + 0.04245*0.04245)}" ixy="0.0" ixz="0.0"
+                 iyy="${(1/12) * 0.0811 * (3*0.022*0.022 + 0.04245*0.04245)}" iyz="0.0"
+                 izz="${0.5 * 0.0811 * 0.022 * 0.022}"/>
+      </inertial>
+    </link>
+    <!-- ===== Joint 5 : 手首ピッチ (X) ===== -->
     <joint name="joint5" type="revolute">
       <parent link="link4"/>
       <child link="link5"/>
-      <origin xyz="0 0 0.04" rpy="0 0 0"/>
-      <axis xyz="0 1 0"/>
-      <limit lower="-2.0" upper="2.0" effort="10.0" velocity="2.0"/>
-      <dynamics damping="20.0" friction="15.0"/>
-    </joint>
-    <!-- Link 5 -->
+      <origin xyz="0 0 0.04245" rpy="0 0 0"/>
+      <axis xyz="1 0 0"/>
+      <limit lower="-1.66" upper="1.66" effort="0.6" velocity="2.2"/>
+      <dynamics damping="0.5" friction="0.2"/>
+    </joint>
     <link name="link5">
       <visual>
-        <origin xyz="0 0 0.02" rpy="0 0 0"/>
-        <geometry>
-          <box size="0.03 0.04 0.04"/>
-        </geometry>
+        <origin xyz="0 0 0.03428" rpy="0 0 0"/>
+        <geometry><box size="0.030 0.036 0.06855"/></geometry>
         <material name="silver"/>
       </visual>
       <collision>
-        <origin xyz="0 0 0.02" rpy="0 0 0"/>
-        <geometry>
-          <box size="0.03 0.04 0.04"/>
-        </geometry>
-      </collision>
-      <inertial>
-        <origin xyz="0 0 0.02" rpy="0 0 0"/>
-        <mass value="0.15"/>
-        <inertia ixx="${(1/12) * 0.15 * (0.04*0.04 + 0.04*0.04)}" ixy="0.0" ixz="0.0"
-                 iyy="${(1/12) * 0.15 * (0.03*0.03 + 0.04*0.04)}" iyz="0.0"
-                 izz="${(1/12) * 0.15 * (0.03*0.03 + 0.04*0.04)}"/>
-      </inertial>
-    </link>
-    <!-- Joint 6 -->
+        <origin xyz="0 0 0.03428" rpy="0 0 0"/>
+        <geometry><box size="0.030 0.036 0.06855"/></geometry>
+      </collision>
+      <inertial>
+        <origin xyz="0.0021 0 0.0394" rpy="0 0 0"/>
+        <mass value="0.0982"/>
+        <inertia ixx="${(1/12) * 0.0982 * (0.036*0.036 + 0.06855*0.06855)}" ixy="0.0" ixz="0.0"
+                 iyy="${(1/12) * 0.0982 * (0.030*0.030 + 0.06855*0.06855)}" iyz="0.0"
+                 izz="${(1/12) * 0.0982 * (0.030*0.030 + 0.036*0.036)}"/>
+      </inertial>
+    </link>
+    <!-- ===== Joint 6 : 手首ロール (Z) ===== -->
     <joint name="joint6" type="revolute">
       <parent link="link5"/>
       <child link="link6"/>
-      <origin xyz="0 0 0.04" rpy="0 0 0"/>
+      <origin xyz="0 0 0.06855" rpy="0 0 0"/>
       <axis xyz="0 0 1"/>
-      <limit lower="-2.0" upper="2.0" effort="10.0" velocity="2.0"/>
-      <dynamics damping="10.0" friction="5.0"/>
-    </joint>
-    <!-- Link 6 -->
+      <limit lower="-3.05" upper="3.05" effort="0.6" velocity="2.2"/>
+      <dynamics damping="0.4" friction="0.15"/>
+    </joint>
     <link name="link6">
       <visual>
-        <origin xyz="0 0 0.01" rpy="0 0 0"/>
-        <geometry>
-          <cylinder radius="0.02" length="0.02"/>
-        </geometry>
+        <origin xyz="0 0 0.0267" rpy="0 0 0"/>
+        <geometry><cylinder radius="0.022" length="0.0534"/></geometry>
         <material name="blue"/>
       </visual>
       <collision>
-        <origin xyz="0 0 0.01" rpy="0 0 0"/>
-        <geometry>
-          <cylinder radius="0.02" length="0.02"/>
-        </geometry>
-      </collision>
-      <inertial>
-        <origin xyz="0 0 0.01" rpy="0 0 0"/>
-        <mass value="0.15"/>
-        <inertia ixx="${(1/12) * 0.15 * (3*0.02*0.02 + 0.02*0.02)}" ixy="0.0" ixz="0.0"
-                 iyy="${(1/12) * 0.15 * (3*0.02*0.02 + 0.02*0.02)}" iyz="0.0"
-                 izz="${0.5 * 0.15 * 0.02 * 0.02}"/>
-      </inertial>
-    </link>
-    <!-- Wrist Camera Joint -->
+        <origin xyz="0 0 0.0267" rpy="0 0 0"/>
+        <geometry><cylinder radius="0.022" length="0.0534"/></geometry>
+      </collision>
+      <inertial>
+        <origin xyz="0 0.0120 0.0368" rpy="0 0 0"/>
+        <mass value="0.1335"/>
+        <inertia ixx="${(1/12) * 0.1335 * (3*0.022*0.022 + 0.0534*0.0534)}" ixy="0.0" ixz="0.0"
+                 iyy="${(1/12) * 0.1335 * (3*0.022*0.022 + 0.0534*0.0534)}" iyz="0.0"
+                 izz="${0.5 * 0.1335 * 0.022 * 0.022}"/>
+      </inertial>
+    </link>
+    <!-- ===== 手首カメラ (ELP基板) =====
+         CAD実測: J6 から (0, +0.03745, +0.0804) m。基板が YZ 平面に立っており
+         光軸は -Y (真横) を向く。ハンドアイとして使う場合は下記 rpy を
+         見直すこと (把持点は +Z 側・カメラより手前にある)。 -->
     <joint name="wrist_camera_joint" type="fixed">
       <parent link="link6"/>
       <child link="wrist_camera_link"/>
-      <origin xyz="0 0.02 0.02" rpy="0 0 0"/>
-    </joint>
-    <!-- Wrist Camera Link -->
+      <origin xyz="0 0.03745 0.0804" rpy="0 0 0"/>
+    </joint>
     <link name="wrist_camera_link">
       <visual>
         <origin xyz="0 0 0" rpy="0 0 0"/>
-        <geometry>
-          <box size="0.01 0.02 0.01"/>
-        </geometry>
+        <geometry><box size="0.024 0.004 0.024"/></geometry>
         <material name="black"/>
       </visual>
-      <collision>
-        <origin xyz="0 0 0" rpy="0 0 0"/>
-        <geometry>
-          <box size="0.01 0.02 0.01"/>
-        </geometry>
-      </collision>
-    </link>
-    <!-- Self collision settings for arm links -->
-    <gazebo reference="link1">
-      <self_collision>false</self_collision>
-    </gazebo>
-    <gazebo reference="link2">
-      <self_collision>false</self_collision>
-    </gazebo>
-    <gazebo reference="link3">
-      <self_collision>false</self_collision>
-    </gazebo>
+    </link>
+    <!-- 光学規約フレーム (Z前方・X右・Y下)。現状の光軸 -Y に対応 -->
+    <joint name="wrist_camera_optical_joint" type="fixed">
+      <parent link="wrist_camera_link"/>
+      <child link="wrist_camera_optical_link"/>
+      <origin xyz="0 0 0" rpy="1.5707963 0 0"/>
+    </joint>
+    <link name="wrist_camera_optical_link"/>
+    <!-- ===== 把持点 / 指先 (IKの目標に使う) =====
+         grasp_link  : 把持面の中心 (J6 から +0.07410) ← MoveIt の目標はここ
+         tcp_link    : 指先端        (J6 から +0.08650) -->
+    <joint name="grasp_joint" type="fixed">
+      <parent link="link6"/>
+      <child link="grasp_link"/>
+      <origin xyz="0 0 0.07410" rpy="0 0 0"/>
+    </joint>
+    <link name="grasp_link"/>
+    <joint name="tcp_joint" type="fixed">
+      <parent link="link6"/>
+      <child link="tcp_link"/>
+      <origin xyz="0 0 0.08650" rpy="0 0 0"/>
+    </joint>
+    <link name="tcp_link"/>
+    <!-- 自己干渉設定 -->
+    <gazebo reference="link1"><self_collision>false</self_collision></gazebo>
+    <gazebo reference="link2"><self_collision>false</self_collision></gazebo>
+    <gazebo reference="link3"><self_collision>false</self_collision></gazebo>
   </xacro:macro>
 </robot>

Commit message: fix: arm mount yaw sign + TRAC-IK solver for reachability
Co-Authored-By: Claude Fable 5 <noreply@anthropic.com>

File: src/amr_description/urdf/amr_robot.urdf.xacro (robot description, xacro)
@@ -83,5 +83,5 @@
     <parent link="base_link"/>
     <child link="arm_base_link"/>
-    <origin xyz="0.15 0 0.075" rpy="0 0 -1.5707963"/>
+    <origin xyz="0.15 0 0.075" rpy="0 0 1.5707963"/>
   </joint>
   <link name="arm_base_link">
