Commit message: fix: reflect hardware fix - camera mast lowered 25mm, drop camera LiDAR sector
Camera mast was lowered 25mm, moving the OAK-D Lite optical center from
(0.182,0.135,0.197) to (0.189,0.135,0.180) [base_footprint frame];
depression angle stays 25deg. Updated oak_d_joint accordingly
(base_link-relative z = 0.180-0.050 = 0.130). Verified via TF:
oak_d_optical_link at (0.1890,0.1350,0.1800), pitch 25.008deg -- matches
spec.

CAD interference analysis confirms the camera housing top (z=0.1997)
now clears the LiDAR scan plane (z=0.210) by 10.3mm, so it no longer
intersects it -- removed the camera self-hit exclusion sector added in
the previous commit (e9883fe), which is no longer needed.

Recomputed the arm exclusion sector from actual joint angles across
home/look_down/grasp/drop_pose rather than the base position alone:
home (all-zero, upright patrol posture) is the worst case since link2
crosses the scan plane there, at the same horizontal position as
arm_base (joint1=0) -- distance 0.310m, bearing -2.40deg, half-angle
4.44deg from link2's cross-section. Other poses' extended links (link3/
link6) stay within this same bearing band. +-1.5deg safety margin ->
sector [-98.34,-86.46]deg = [-1.7164,-1.5090]rad in the LiDAR's own
scan-angle frame, matching the given target values exactly. Range
cutoff unchanged (0.60m).

Co-Authored-By: Claude Sonnet 5 <noreply@anthropic.com>

File: src/amr_description/urdf/amr_robot.urdf.xacro (robot description, xacro)
@@ -40,13 +40,16 @@
   <xacro:include filename="base_omni_4wheel.xacro"/>
   <xacro:base_omni_4wheel/>
-  <!-- 2026-08-24 実機HW確定: OAK-D Lite 光学中心 (0.182, 0.135, 0.197)
-       [base_footprint基準]、俯角25°。oak_d_optical_joint(下記、Z前方の
-       光学フレーム規約)は並進0のため、oak_d_link原点=光学中心の絶対位置
-       をそのままbase_link基準に変換すればよい: z = 0.197 - 0.050 = 0.147。
-       pitch = 25° = 0.4363323 rad(既存符号規約=正のpitchで下向きを踏襲)。 -->
+  <!-- 2026-09-01 ハード修正反映: カメラマストを25mm下げた結果、OAK-D Lite
+       光学中心が (0.182, 0.135, 0.197) → (0.189, 0.135, 0.180)
+       [base_footprint基準] に変更。俯角25°は変更なし。
+       oak_d_optical_joint(下記、Z前方の光学フレーム規約)は並進0のため、
+       oak_d_link原点=光学中心の絶対位置をそのままbase_link基準に変換
+       すればよい: z = 0.180 - 0.050 = 0.130。
+       pitch = 25° = 0.4363323 rad(既存符号規約=正のpitchで下向きを踏襲、
+       角度自体は変更なし)。 -->
   <joint name="oak_d_joint" type="fixed">
     <parent link="base_link"/>
     <child link="oak_d_link"/>
-    <origin xyz="0.182 0.135 0.147" rpy="0 0.4363323 0"/>
+    <origin xyz="0.189 0.135 0.130" rpy="0 0.4363323 0"/>
   </joint>
   <link name="oak_d_link">
